Commit message: calib board

File: simulation/urdf/gp4.xacro (robot description, xacro)
@@ -244,5 +244,5 @@
     </inertial>
       <visual>
-        <origin xyz="0 0 0" rpy="0 0 0"/>
+        <origin xyz="0 0 0" rpy="0 0 ${-21.0/180.0*pi}"/>
         <geometry>
           <mesh filename="file://$(find gp4_lego)/simulation/meshes/robot/tool_base.stl"/>
@@ -302,10 +302,10 @@
     </joint>
     <joint name="link_6_fts" type="fixed">
-      <origin xyz="${0.0437/2} 0 0" rpy="0 ${pi/2.0} 0" />
+      <origin xyz="${0.0445/2} 0 0" rpy="0 ${pi/2.0} 0" />
       <parent link="flange" />
       <child link="fts" />
     </joint>
     <joint name="fts_tool" type="revolute">
-      <origin xyz="0 0 ${0.0437/2}" rpy="0 0 ${pi}" />
+      <origin xyz="0 0 ${0.0445/2}" rpy="0 0 ${pi}" />
       <parent link="fts" />
       <child link="link_tool" />

Commit message: update gp4 model

File: simulation/urdf/gp4.xacro (robot description, xacro)
@@ -302,10 +302,10 @@
     </joint>
     <joint name="link_6_fts" type="fixed">
-      <origin xyz="${0.0437/2} 0 0" rpy="0 ${pi/2.0} 0" />
+      <origin xyz="${0.0445/2} 0 0" rpy="0 ${pi/2.0} 0" />
       <parent link="flange" />
       <child link="fts" />
     </joint>
     <joint name="fts_tool" type="revolute">
-      <origin xyz="0 0 ${0.0437/2}" rpy="0 0 ${pi}" />
+      <origin xyz="0 0 ${0.0445/2}" rpy="0 0 ${pi}" />
       <parent link="fts" />
       <child link="link_tool" />

Commit message: live sim

File: simulation/urdf/gp4.xacro (robot description, xacro)
@@ -302,10 +302,10 @@
     </joint>
     <joint name="link_6_fts" type="fixed">
-      <origin xyz="${0.0445/2} 0 0" rpy="0 ${pi/2.0} 0" />
+      <origin xyz="${0.0395/2} 0 0" rpy="0 ${pi/2.0} 0" />
       <parent link="flange" />
       <child link="fts" />
     </joint>
     <joint name="fts_tool" type="revolute">
-      <origin xyz="0 0 ${0.0445/2}" rpy="0 0 ${pi}" />
+      <origin xyz="0 0 ${0.0395/2}" rpy="0 0 ${pi}" />
       <parent link="fts" />
       <child link="link_tool" />

Commit message: update eoat dim

File: simulation/urdf/gp4.xacro (robot description, xacro)
@@ -302,10 +302,10 @@
     </joint>
     <joint name="link_6_fts" type="fixed">
-      <origin xyz="${0.0395/2} 0 0" rpy="0 ${pi/2.0} 0" />
+      <origin xyz="${0.0505/2} 0 0" rpy="0 ${pi/2.0} 0" />
       <parent link="flange" />
       <child link="fts" />
     </joint>
     <joint name="fts_tool" type="revolute">
-      <origin xyz="0 0 ${0.0395/2}" rpy="0 0 ${pi}" />
+      <origin xyz="0 0 ${0.0505/2}" rpy="0 0 ${pi}" />
       <parent link="fts" />
       <child link="link_tool" />
